File: designs/Pufferfish-Interface-2/Pufferfish-Interface-2 -1.kicad_pcb (KiCad board)
At the start: 2 copper layers, 76.2 x 57.1 mm, 79 parts, among them J1 Conn_01x09_Male, Q1 2N7002E, Q10 2N7002E, Q2 2N7002E, Q3 2N7002E, Q4 2N7002E, Q5 DMN10H220L, Q6 DMN10H220L, Q7 DMN10H220L, Q8 2N7002E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

Commit message: assembly changes (footprint, etc)
Routing:
- net Net-(BUZZ1-Pad2): track 17.3 -> 27.1 mm
- net Net-(BUZZ1-Pad3): track 27.9 -> 29.7 mm, vias 1 -> 0
Changed lines of the file:
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@@
     (thickness 1.6)
     (drawings 8)
-    (tracks 560)
+    (tracks 558)
     (zones 0)
     (modules 79)
@@
   (layers
     (0 F.Cu signal)
-    (31 B.Cu signal)
-    (32 B.Adhes user)
+    (31 B.Cu signal hide)
+    (32 B.Adhes user hide)
     (33 F.Adhes user)
-    (34 B.Paste user)
+    (34 B.Paste user hide)
     (35 F.Paste user)
-    (36 B.SilkS user)
+    (36 B.SilkS user hide)
     (37 F.SilkS user)
-    (38 B.Mask user)
+    (38 B.Mask user hide)
     (39 F.Mask user)
     (40 Dwgs.User user)
@@
     (46 B.CrtYd user)
     (47 F.CrtYd user)
-    (48 B.Fab user)
+    (48 B.Fab user hide)
     (49 F.Fab user)
   )
@@
     (add_net GND)
   )
-  (module Pufferfish:Buzzer-MSS5MMG (layer F.Cu)
-    (at 16.002 39.37)
-    (descr "Medical regulatory buzzer")
-    (fp_text reference BUZZ1 (at -4.90728 12.3063) (layer F.SilkS)
-      (effects (font (size 1 1) (thickness 0.15)))
-    )
-    (fp_text value BUZZER-MALLORY (at 0 13) (layer F.Fab)
-      (effects (font (size 1 1) (thickness 0.15)))
-    )
-    (fp_circle (center 0 0) (end 11.5 0) (layer F.SilkS) (width 0.2032))
-    (pad 2 thru_hole circle (at -4.9 5.4) (size 1.6 1.6) (drill 1) (layers *.Cu *.Mask)
-      (net 4 "Net-(BUZZ1-Pad2)"))
-    (pad 3 thru_hole circle (at -4.9 2.9) (size 1.6 1.6) (drill 1) (layers *.Cu *.Mask)
-      (net 3 "Net-(BUZZ1-Pad3)"))
-    (pad 1 thru_hole circle (at -7.5 0) (size 1.6 1.6) (drill 1) (layers *.Cu *.Mask)
-      (net 2 5V))
-    (pad 4 thru_hole circle (at 7.5 0) (size 1.6 1.6) (drill 1) (layers *.Cu *.Mask)
-      (net 1 "Net-(BUZZ1-Pad4)"))
-  )
   (module Pufferfish:STANDOFF-ELECTRICAL-NOTHERMALS (layer F.Cu)
     (at 64.77 6.35)
@@
     )
   )
+  (module Pufferfish:Buzzer-MSS5MMG (layer F.Cu)
+    (at 16.002 39.37)
+    (descr "Medical regulatory buzzer")
+    (fp_text reference BUZZ1 (at -4.90728 12.3063) (layer F.SilkS)
+      (effects (font (size 1 1) (thickness 0.15)))
+    )
+    (fp_text value BUZZER-MALLORY (at 0 13) (layer F.Fab)
+      (effects (font (size 1 1) (thickness 0.15)))
+    )
+    (fp_circle (center 0 0) (end 11.5 0) (layer F.SilkS) (width 0.2032))
+    (pad 4 thru_hole circle (at 7.5 0) (size 1.6 1.6) (drill 1) (layers *.Cu *.Mask)
+      (net 1 "Net-(BUZZ1-Pad4)"))
+    (pad 1 thru_hole circle (at -7.5 0) (size 1.6 1.6) (drill 1) (layers *.Cu *.Mask)
+      (net 2 5V))
+    (pad 3 thru_hole circle (at 4.9 2.9) (size 1.6 1.6) (drill 1) (layers *.Cu *.Mask)
+      (net 3 "Net-(BUZZ1-Pad3)"))
+    (pad 2 thru_hole circle (at 4.9 5.4) (size 1.6 1.6) (drill 1) (layers *.Cu *.Mask)
+      (net 4 "Net-(BUZZ1-Pad2)"))
+  )
   (module Pufferfish:CAP_SMD_0805 (layer F.Cu)
     (at 51.1325 21.336)
@@
   (segment (start 17.24454 28.448) (end 19.08048 26.61206) (width 0.508) (layer F.Cu) (net 2))
   (segment (start 14.313682 28.448) (end 17.24454 28.448) (width 0.508) (layer F.Cu) (net 2))
+  (segment (start 21.066 42.106) (end 20.902 42.27) (width 0.25) (layer B.Cu) (net 3))
+  (segment (start 21.066 33.02) (end 21.066 42.106) (width 0.25) (layer B.Cu) (net 3))
+  (segment (start 7.472 42.27) (end 20.902 42.27) (width 0.25) (layer F.Cu) (net 3))
   (segment (start 2.54 37.338) (end 7.472 42.27) (width 0.25) (layer F.Cu) (net 3))
-  (segment (start 7.472 42.27) (end 11.102 42.27) (width 0.25) (layer F.Cu) (net 3))
-  (via (at 21.066 38.9349) (size 0.8) (drill 0.4) (layers F.Cu B.Cu) (net 3))
-  (segment (start 17.7309 42.27) (end 21.066 38.9349) (width 0.25) (layer F.Cu) (net 3))
-  (segment (start 11.102 42.27) (end 17.7309 42.27) (width 0.25) (layer F.Cu) (net 3))
-  (segment (start 21.066 33.02) (end 21.066 38.9349) (width 0.25) (layer B.Cu) (net 3))
   (segment (start 13.192 48.244) (end 18.542 53.594) (width 0.25) (layer B.Cu) (net 4))
   (segment (start 12.192 48.244) (end 13.192 48.244) (width 0.25) (layer B.Cu) (net 4))
+  (segment (start 9.078 44.77) (end 20.902 44.77) (width 0.25) (layer B.Cu) (net 4))
   (segment (start 8.382 45.466) (end 9.078 44.77) (width 0.25) (layer B.Cu) (net 4))
   (segment (start 11.526 48.26) (end 9.906 48.26) (width 0.25) (layer B.Cu) (net 4))
@@
   (segment (start 9.906 48.26) (end 8.382 46.736) (width 0.25) (layer B.Cu) (net 4))
   (segment (start 11.542 48.244) (end 11.526 48.26) (width 0.25) (layer B.Cu) (net 4))
-  (segment (start 9.078 44.77) (end 11.102 44.77) (width 0.25) (layer B.Cu) (net 4))
   (via (at 28.55722 24.98598) (size 0.8) (drill 0.4) (layers F.Cu B.Cu) (net 5))
   (segment (start 36.7515 23.6265) (end 36.248 24.13) (width 0.25) (layer F.Cu) (net 5))
